File: kicad/clock-radio.kicad_pcb (KiCad board)
At the start: 4 copper layers, 32.3 x 31.8 mm, 53 parts, among them J1 Rotary Encoder Header, J2 Antenna, J3 USB_C_Receptacle_USB2.0_16P, J4 SWD Header, J5 Display Header, J6 Speaker Header, J7 Coin Cell, SW1 BOOT0, U1 DS3231MZ, U2 STM32G0B1CETx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

Commit message: updated cap
Parts:
- C19: value 470u -> 1u
Changed lines of the file:
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@@
 			(drillshape 0)
 			(scaleselection 1)
-			(outputdirectory "/home/bbuckham/Downloads/")
+			(outputdirectory "../clock-radio gerber/update/")
 		)
 	)
@@
 			)
 		)
-		(property "Value" "470u"
+		(property "Value" "1u"
 			(at 0 -1.16 90)
 			(layer "B.Fab")
